File: on_air.kicad_pcb (KiCad board)
At the start: 2 copper layers, 15 parts, among them Q1 NPN, Q2 NPN, Q3 PNP

Commit message: B.Cu
Parts:
- Q1, Q2: footprint Package_TO_SOT_THT:TO-92 -> Elopin:NPN_THT
- Q3: footprint Package_TO_SOT_THT:TO-92 -> Elopin:PNP_THT
- moved D3 93.1 mm to (39.0, 42.5), turned to -90 degrees
- moved 3xAA1 67.0 mm to (125.6, 28.5), turned to 0 degrees
- moved D2 57.3 mm to (73.7, 42.5), turned to -90 degrees
- moved Q1 55.4 mm to (33.0, 31.5), turned to 90 degrees
- moved R6 55.1 mm to (100.0, 30.0), turned to -90 degrees
- moved R2 42.8 mm to (25.5, 25.2), turned to -90 degrees
- moved Q3 32.6 mm to (85.0, 46.5), turned to -90 degrees
- moved R4 29.8 mm to (75.5, 25.2), turned to -90 degrees
- moved R1 27.4 mm to (40.5, 25.2), turned to -90 degrees
- moved R5 26.6 mm to (94.5, 39.2), turned to -90 degrees
- moved D1 26.3 mm to (103.7, 42.5), turned to -90 degrees
- moved C2 24.1 mm to (59.8, 33.0), turned to 0 degrees
- moved C1 22.3 mm to (62.5, 38.5), turned to 180 degrees
- moved Q2 22.2 mm to (93.5, 31.5), turned to 90 degrees
- moved R3 18.9 mm to (69.0, 25.2), turned to -90 degrees
Routing:
- net Net-(D1-K): track 36.0 -> 71.1 mm
- net Net-(3xAA1-+): track 127.2 -> 157.5 mm
- net Net-(D1-A): track 37.9 -> 65.3 mm
- net Net-(Q1-B): track 21.2 -> 38.9 mm
- net Net-(Q3-B): track 26.9 -> 9.71 mm
- net Net-(Q2-C): track 55.5 -> 42.1 mm
- net Net-(Q2-B): track 19.2 -> 30.4 mm
- net Net-(Q1-C): track 37.0 -> 26.0 mm
- net Net-(3xAA1--): track 98.5 -> 91.7 mm
- added copper zone on B.Cu, net (none)
Other:
- board outline added: 110 x 45 mm
